Commit message: created launch files: for empty gazebo world and for custom gazebo world

File: urdf/autonomous_robot.urdf (robot description, URDF)
Before this commit: robot autonomous_robot, 2 links, 1 joints
Links:
- added link caster_wheel, mass ${mass_caster}; collision sphere radius=${caster_radius}; visual sphere radius=${caster_radius}
- added link left_wheel, mass ${mass_wheel}; collision cylinder length=${d} radius=${r}; visual cylinder length=${d} radius=${r}
- added link right_wheel, mass ${mass_wheel}; collision cylinder length=${d} radius=${r}; visual cylinder length=${d} radius=${r}
Joints:
- added joint base_caster_wheel_joint: type fixed, parent base_link, child caster_wheel, origin xyz=-0.15 0 -0.05 rpy=0 0 0
- added joint base_left_wheel_joint: type continuous, parent base_link, child left_wheel, origin xyz=0.15 0.175 0 rpy=0 0 0, axis 0 1 0
- added joint base_right_wheel_joint: type continuous, parent base_link, child right_wheel, origin xyz=0.15 -0.175 0 rpy=0 0 0, axis 0 1 0

Commit message: added lidar scan link to the robot

File: urdf/autonomous_robot.urdf (robot description, URDF)
Before this commit: robot autonomous_robot, 5 links, 4 joints
Links:
- added link scan_link, mass 0.1; collision cylinder length=0.025 radius=0.1; visual cylinder length=0.025 radius=0.1
- added link support_link; visual box size=0.2 0.2 0.05
Joints:
- added joint lidar_support_joint: type fixed, parent base_link, child support_link, origin xyz=0 0 0.075 rpy=0 0 0
- added joint scan_joint: type fixed, parent support_link, child scan_link, origin xyz=0 0 0.0375 rpy=0 0 0, axis 0 1 0

Commit message: added camera to the robot

File: urdf/autonomous_robot.urdf (robot description, URDF)
Before this commit: robot autonomous_robot, 7 links, 6 joints
Links:
- added link camera_link, mass 0.1; collision box size=0.03 0.03 0.03; visual box size=0.03 0.03 0.03
- added link camera_link_optical
Joints:
- added joint camera_joint: type fixed, parent base_link, child camera_link, origin xyz=0.18 0 0.065 rpy=0 0 0, axis 0 1 0
- added joint camera_optical_joint: type fixed, parent camera_link, child camera_link_optical, origin xyz=0 0 0 rpy=-1.5707 0 -1.5707

Commit message: updated urdf model

File: urdf/autonomous_robot.urdf (robot description, URDF)
Before this commit: robot autonomous_robot, 9 links, 8 joints
Links:
- removed link support_link
- link scan_link: geometry collision cylinder length=0.025 radius=0.1; visual cylinder length=0.05 radius=0.1
Joints:
- removed joint lidar_support_joint
- joint base_caster_wheel_joint: origin xyz=-0.15 0 -0.05 rpy=0 0 0 -> xyz=-0.15 0 -0.1 rpy=0 0 0
- joint base_left_wheel_joint: origin xyz=0.15 0.175 0 rpy=0 0 0 -> xyz=0.15 0.175 -0.05 rpy=0 0 0
- joint base_right_wheel_joint: origin xyz=0.15 -0.175 0 rpy=0 0 0 -> xyz=0.15 -0.175 -0.05 rpy=0 0 0
- joint camera_joint: origin xyz=0.18 0 0.065 rpy=0 0 0 -> xyz=0.2 0 0 rpy=0 0 0
- joint scan_joint: origin xyz=0 0 0.0375 rpy=0 0 0 -> xyz=0 0 0.1 rpy=0 0 0; parent support_link -> base_link

Commit message: working with robot, trying to use rtab map

File: urdf/autonomous_robot.urdf (robot description, URDF)
Before this commit: robot autonomous_robot, 8 links, 7 joints
Links:
- added link support_link, mass 0.1; collision box size=0.2 0.2 0.05; visual box size=0.2 0.2 0.05
- link scan_link: geometry collision cylinder length=0.025 radius=0.1; visual cylinder length=0.02 radius=0.1
Joints:
- added joint lidar_support_joint: type fixed, parent base_link, child support_link, origin xyz=0 0 0.1 rpy=0 0 0
- joint camera_joint: origin xyz=0.2 0 0 rpy=0 0 0 -> xyz=0.18 0 0.09 rpy=0 0 0
- joint scan_joint: origin xyz=0 0 0.1 rpy=0 0 0 -> xyz=0 0 0.135 rpy=0 0 0
